File: Kicad/NiController/ledRing.kicad_sch (KiCad schematic)
At the start: 32 parts

Commit message: led ring 4
Parts:
- renumbered C2101 to C201, C2102 to C202, C2103 to C203, C2104 to C204, C2105 to C205, C2106 to C206, C2107 to C207, C2108 to C208, C2109 to C209, C2110 to C210, C2111 to C211, C2112 to C212, C2113 to C213, C2114 to C214, C2115 to C215, C2116 to C216, D2101 to D201, D2102 to D202, D2103 to D203, D2104 to D204, D2105 to D205, D2106 to D206, D2107 to D207, D2108 to D208, D2109 to D209, D2110 to D210, D2111 to D211, D2112 to D212, D2113 to D213, D2114 to D214, D2115 to D215, D2116 to D216
