File: Kicad/NiController/ledRing4.kicad_sch (KiCad schematic)
At the start: 6 parts

Commit message: led ring 4
Parts:
- removed H? (x4): MountingHole_Pad, MountingHole:MountingHole_2.5mm_Pad_Via, symbol Mechanical:MountingHole_Pad
- gave numbers to parts that had none: 2
