File: Kicad/NiController/encoder4button4.kicad_sch (KiCad schematic)
At the start: 7 parts, among them J3801 Conn_02x09_Counter_Clockwise, J3802 Conn_02x03_Odd_Even, J3803 Conn_02x03_Odd_Even

Commit message: enc4btn4
Parts:
- removed J3801: Conn_02x09_Counter_Clockwise, symbol Connector_Generic:Conn_02x09_Counter_Clockwise
- added J1001: Conn_02x10_Odd_Even, Connector_IDC:IDC-Header_2x10_P2.54mm_Vertical, symbol Connector_Generic:Conn_02x10_Odd_Even
- J3802: footprint Connector_PinHeader_2.54mm:PinHeader_2x03_P2.54mm_Vertical -> Connector_IDC:IDC-Header_2x03_P2.54mm_Vertical
Connections:
- net 0_GPA0: now also J1001.3 (Pin_3)
- net 0_GPA1: now also J1001.5 (Pin_5)
- net 0_GPA2: now also J1001.7 (Pin_7)
- net 0_GPA3: now also J1001.9 (Pin_9)
- net 0_GPA4: now also J1001.11 (Pin_11)
- net 0_GPA5: now also J1001.13 (Pin_13)
- net 0_GPA6: now also J1001.15 (Pin_15)
- net 0_GPA7: now also J1001.17 (Pin_17)
- net 0_GPB0: now also J1001.18 (Pin_18)
- net 0_GPB1: now also J1001.16 (Pin_16)
- net 0_GPB2: now also J1001.14 (Pin_14)
- net 0_GPB3: now also J1001.12 (Pin_12)
- net 0_GPB4: now also J1001.10 (Pin_10)
- net 0_GPB5: now also J1001.8 (Pin_8)
- net 0_GPB6: now also J1001.6 (Pin_6)
- net 0_GPB7: now also J1001.4 (Pin_4)
- net GND: now also J1001.1 (Pin_1), J1001.19 (Pin_19), J1001.2 (Pin_2), J1001.20 (Pin_20)
Other:
- sheet button9 renamed button3
- sheet encoder9 renamed encoder3
- added sheet button0 (button.kicad_sch)
- added sheet button1 (button.kicad_sch)
- added sheet button2 (button.kicad_sch)
- added sheet encoder0 (encoder.kicad_sch)
- added sheet encoder1 (encoder.kicad_sch)
- added sheet encoder2 (encoder.kicad_sch)

Commit message: enc btn
Parts:
- removed J3803: Conn_02x03_Odd_Even, Connector_PinHeader_2.54mm:PinHeader_2x03_P2.54mm_Vertical, symbol Connector_Generic:Conn_02x03_Odd_Even
- added J1002, J1003: Conn_01x03, Connector_PinSocket_2.54mm:PinSocket_1x03_P2.54mm_Vertical, symbol Connector_Generic:Conn_01x03
Connections:
- net GND: now also J1002.1 (Pin_1), J1003.1 (Pin_1)
- net LED_5V: now also J1002.3 (Pin_3), J1003.3 (Pin_3)
- net LED_DIN: now also J1002.2 (Pin_2)
- net LED_RING_DOUT: now also J1003.2 (Pin_2)
Changed lines of the file:
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@@
 	(wire
 		(pts
-			(xy 52.705 128.905) (xy 60.325 128.905)
+			(xy 50.8 142.875) (xy 58.42 142.875)
 		)
 		(stroke
@@
 	(wire
 		(pts
-			(xy 60.325 128.905) (xy 60.325 131.445)
+			(xy 58.42 142.875) (xy 58.42 145.415)
 		)
 		(stroke
@@
 	)
 	(label "LED_5V"
-		(at 52.705 133.985 0)
+		(at 50.8 147.955 0)
 		(effects
 			(font
@@
 	)
 	(label "LED_RING_DOUT"
-		(at 52.705 131.445 0)
+		(at 50.8 145.415 0)
 		(effects
 			(font
@@
 	)
 	(symbol
-		(lib_id "Connector_Generic:Conn_02x03_Odd_Even")
-		(at 45.085 131.445 0)
+		(lib_id "power:GND")
+		(at 58.42 145.415 0)
 		(unit 1)
 		(exclude_from_sim no)
@@
 		(dnp no)
 		(fields_autoplaced yes)
-		(property "Reference" "J3803"
-			(at 46.355 122.555 0)
-			(effects
-				(font
-					(size 1.27 1.27)
-				)
-			)
-		)
-		(property "Value" "Conn_02x03_Odd_Even"
-			(at 46.355 125.095 0)
-			(effects
-				(font
-					(size 1.27 1.27)
-				)
-			)
-		)
-		(property "Footprint" "Connector_PinHeader_2.54mm:PinHeader_2x03_P2.54mm_Vertical"
-			(at 45.085 131.445 0)
-			(effects
-				(font
-					(size 1.27 1.27)
-				)
-				(hide yes)
-			)
-		)
-		(property "Datasheet" "~"
-			(at 45.085 131.445 0)
-			(effects
-				(font
-					(size 1.27 1.27)
-				)
-				(hide yes)
-			)
-		)
-		(property "Description" "Generic connector, double row, 02x03, odd/even pin numbering scheme (row 1 odd numbers, row 2 even numbers), script generated (kicad-library-utils/schlib/autogen/connector/)"
-			(at 45.085 131.445 0)
-			(effects
-				(font
-					(size 1.27 1.27)
-				)
-				(hide yes)
-			)
-		)
-		(pin "3"
-		)
-		(pin "1"
-		)
-		(pin "5"
-		)
-		(pin "2"
-		)
-		(pin "4"
-		)
-		(pin "6"
-		)
-		(instances
-			(project "NiController"
-				(path "/e70b5343-6e83-46b0-b96e-745e0612c526/2a4c6518-6eed-4a25-9459-9f6a8208ccfc"
-					(reference "J3803")
-					(unit 1)
-				)
-			)
-		)
-	)
-	(symbol
-		(lib_id "power:GND")
-		(at 60.325 131.445 0)
-		(unit 1)
-		(exclude_from_sim no)
-		(in_bom yes)
-		(on_board yes)
-		(dnp no)
-		(fields_autoplaced yes)
 		(property "Reference" "#PWR03805"
-			(at 60.325 137.795 0)
+			(at 58.42 151.765 0)
 			(effects
 				(font
@@
 		)
 		(property "Value" "GND"
-			(at 60.325 136.525 0)
+			(at 58.42 150.495 0)
 			(effects
 				(font
@@
 		)
 		(property "Footprint" ""
-			(at 60.325 131.445 0)
+			(at 58.42 145.415 0)
 			(effects
 				(font
@@
 		)
 		(property "Datasheet" ""
-			(at 60.325 131.445 0)
+			(at 58.42 145.415 0)
 			(effects
 				(font
@@
 		)
 		(property "Description" "Power symbol creates a global label with name \"GND\" , ground"
-			(at 60.325 131.445 0)
+			(at 58.42 145.415 0)
 			(effects
 				(font
@@
 	)
 	(symbol
+		(lib_id "Connector_Generic:Conn_01x03")
+		(at 45.72 145.415 0)
+		(mirror y)
+		(unit 1)
+		(exclude_from_sim no)
+		(in_bom yes)
+		(on_board yes)
+		(dnp no)
+		(property "Reference" "J1003"
+			(at 42.545 144.1449 0)
+			(effects
+				(font
+					(size 1.27 1.27)
+				)
+				(justify left)
+			)
+		)
+		(property "Value" "Conn_01x03"
+			(at 42.545 146.6849 0)
+			(effects
+				(font
+					(size 1.27 1.27)
+				)
+				(justify left)
+			)
+		)
+		(property "Footprint" "Connector_PinSocket_2.54mm:PinSocket_1x03_P2.54mm_Vertical"
+			(at 45.72 145.415 0)
+			(effects
+				(font
+					(size 1.27 1.27)
+				)
+				(hide yes)
+			)
+		)
+		(property "Datasheet" "~"
+			(at 45.72 145.415 0)
+			(effects
+				(font
+					(size 1.27 1.27)
+				)
+				(hide yes)
+			)
+		)
+		(property "Description" "Generic connector, single row, 01x03, script generated (kicad-library-utils/schlib/autogen/connector/)"
+			(at 45.72 145.415 0)
+			(effects
+				(font
+					(size 1.27 1.27)
+				)
+				(hide yes)
+			)
+		)
+		(pin "1"
+		)
+		(pin "2"
+		)
+		(pin "3"
+		)
+		(instances
+			(project ""
+				(path "/e70b5343-6e83-46b0-b96e-745e0612c526/2a4c6518-6eed-4a25-9459-9f6a8208ccfc"
+					(reference "J1003")
+					(unit 1)
+				)
+			)
+		)
+	)
+	(symbol
 		(lib_id "Mechanical:MountingHole_Pad")
 		(at 133.35 50.8 0)
@@
 	)
 	(symbol
+		(lib_id "Connector_Generic:Conn_01x03")
+		(at 45.085 131.445 0)
+		(unit 1)
+		(exclude_from_sim no)
+		(in_bom yes)
+		(on_board yes)
+		(dnp no)
+		(fields_autoplaced yes)
+		(property "Reference" "J1002"
+			(at 48.26 130.1749 0)
+			(effects
+				(font
+					(size 1.27 1.27)
+				)
+				(justify left)
+			)
+		)
+		(property "Value" "Conn_01x03"
+			(at 48.26 132.7149 0)
+			(effects
+				(font
+					(size 1.27 1.27)
+				)
+				(justify left)
+			)
+		)
+		(property "Footprint" "Connector_PinSocket_2.54mm:PinSocket_1x03_P2.54mm_Vertical"
+			(at 45.085 131.445 0)
+			(effects
+				(font
+					(size 1.27 1.27)
+				)
+				(hide yes)
+			)
+		)
+		(property "Datasheet" "~"
+			(at 45.085 131.445 0)
+			(effects
+				(font
+					(size 1.27 1.27)
+				)
+				(hide yes)
+			)
+		)
+		(property "Description" "Generic connector, single row, 01x03, script generated (kicad-library-utils/schlib/autogen/connector/)"
+			(at 45.085 131.445 0)
+			(effects
+				(font
+					(size 1.27 1.27)
+				)
+				(hide yes)
+			)
+		)
+		(pin "1"
+		)
+		(pin "2"
+		)
+		(pin "3"
+		)
+		(instances
+			(project ""
+				(path "/e70b5343-6e83-46b0-b96e-745e0612c526/2a4c6518-6eed-4a25-9459-9f6a8208ccfc"
+					(reference "J1002")
+					(unit 1)
+				)
+			)
+		)
+	)
+	(symbol
 		(lib_id "Connector_Generic:Conn_02x10_Odd_Even")
 		(at 43.18 35.56 0)
@@
 		)
 		(instances
-			(project "NiController"
+			(project "NiController_encoder4button4"
 				(path "/e70b5343-6e83-46b0-b96e-745e0612c526/2a4c6518-6eed-4a25-9459-9f6a8208ccfc"
 					(page "6")
@@
 		)
 		(instances
-			(project "NiController"
+			(project "NiController_encoder4button4"
 				(path "/e70b5343-6e83-46b0-b96e-745e0612c526/2a4c6518-6eed-4a25-9459-9f6a8208ccfc"
 					(page "5")
@@
 		)
 		(instances
-			(project "NiController"
+			(project "NiController_encoder4button4"
 				(path "/e70b5343-6e83-46b0-b96e-745e0612c526/2a4c6518-6eed-4a25-9459-9f6a8208ccfc"
 					(page "4")
@@
 		)
 		(instances
-			(project "NiController"
+			(project "NiController_encoder4button4"
 				(path "/e70b5343-6e83-46b0-b96e-745e0612c526/2a4c6518-6eed-4a25-9459-9f6a8208ccfc"
 					(page "19")
@@
 		)
 		(instances
-			(project "NiController"
+			(project "NiController_encoder4button4"
 				(path "/e70b5343-6e83-46b0-b96e-745e0612c526/2a4c6518-6eed-4a25-9459-9f6a8208ccfc"
 					(page "9")
@@
 		)
 		(instances
-			(project "NiController"
+			(project "NiController_encoder4button4"
 				(path "/e70b5343-6e83-46b0-b96e-745e0612c526/2a4c6518-6eed-4a25-9459-9f6a8208ccfc"
 					(page "8")
@@
 		)
 		(instances
-			(project "NiController"
+			(project "NiController_encoder4button4"
 				(path "/e70b5343-6e83-46b0-b96e-745e0612c526/2a4c6518-6eed-4a25-9459-9f6a8208ccfc"
 					(page "7")
@@
 		)
 		(instances
-			(project "NiController"
+			(project "NiController_encoder4button4"
 				(path "/e70b5343-6e83-46b0-b96e-745e0612c526/2a4c6518-6eed-4a25-9459-9f6a8208ccfc"
 					(page "29")
