File: Kicad/NiController/NiController_encoder4button4.kicad_pcb (KiCad board)
At the start: 2 copper layers, 100 x 100 mm, 39 parts, among them J1001 Conn_02x10_Odd_Even, J3802 Conn_02x03_Odd_Even, J3803 Conn_02x03_Odd_Even, SW1901 SW_Push, SW2901 SW_Push, SW401 RotaryEncoder_Switch, SW501 RotaryEncoder_Switch, SW601 RotaryEncoder_Switch, SW701 RotaryEncoder_Switch, SW801 SW_Push, SW901 SW_Push

Commit message: enc btn
Parts:
- removed J3803: Conn_02x03_Odd_Even, Connector_PinHeader_2.54mm:PinHeader_2x03_P2.54mm_Vertical
- added J1002: Conn_01x03, Connector_PinSocket_2.54mm:PinSocket_1x03_P2.54mm_Vertical, F.Cu at (104.1, 99.1)
- added J1003: Conn_01x03, Connector_PinSocket_2.54mm:PinSocket_1x03_P2.54mm_Vertical, F.Cu at (149.9, 99.1)
- moved H3801 128.4 mm to (105.0, 174.0)
- moved H3802 113.6 mm to (149.0, 174.0)
- moved H3804 45.6 mm to (105.0, 80.0)
- moved C1901 30.7 mm to (114.5, 173.0), turned to 0 degrees
- moved C801 30.7 mm to (114.5, 148.0), turned to 0 degrees
- moved C2901 30.3 mm to (139.5, 173.0)
- moved C901 30.3 mm to (139.5, 148.0), turned to 0 degrees
- moved C501 27.7 mm to (139.5, 100.0)
- moved C701 27.7 mm to (139.5, 125.0)
- moved C502 27.7 mm to (142.0, 100.0)
- moved C702 27.7 mm to (142.0, 125.0)
- moved C1902 26.0 mm to (120.0, 156.5)
- moved C802 26.0 mm to (120.0, 131.5)
- moved C403 25.6 mm to (112.0, 100.0)
- moved C603 25.6 mm to (112.0, 125.0), turned to -90 degrees
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Routing:
- net /encoder4button4/LED_5V: track 0.00 -> 197.5 mm
- net /encoder4button4/LED_DOUT: track 0.00 -> 97.2 mm
- net /encoder4button4/LED_RING_DOUT: track 0.00 -> 72.0 mm, vias 0 -> 1
- net /encoder4button4/button1/DOUT: track 0.00 -> 50.1 mm
- net /encoder4button4/LED_DIN: track 0.00 -> 26.4 mm
- net /encoder4button4/button2/DOUT: track 0.00 -> 23.8 mm
- net /encoder4button4/button0/DOUT: track 0.00 -> 23.6 mm
- net /encoder4button4/0_GPB3: track 39.7 -> 30.7 mm
- net /encoder4button4/0_GPA6: track 31.1 -> 36.8 mm
- net /encoder4button4/0_GPB1: track 19.9 -> 23.4 mm
- net /encoder4button4/0_GPA5: track 57.8 -> 54.6 mm, vias 0 -> 2
- net /encoder4button4/0_GPA7: track 34.2 -> 30.9 mm
- net /encoder4button4/0_GPA3: track 33.0 -> 34.6 mm, vias 0 -> 2
- net /encoder4button4/0_GPA4: track 37.6 -> 39.1 mm, vias 0 -> 2
- net /encoder4button4/0_GPB2: track 21.0 -> 22.0 mm
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- added copper zone on B.Cu, net GND
- added copper zone on F.Cu, net GND
Other:
- board size 100 x 100 mm -> 50 x 100 mm

Commit message: main
Parts:
- SW401, SW501, SW601, SW701: footprint Rotary_Encoder:RotaryEncoder_Bourns_Vertical_PEC12R-3x17F-Sxxxx -> NiLibrary:PEC11-4xxxF-Sxxxx
- moved SW401 7.91 mm to (114.5, 89.5), turned to 0 degrees
- moved SW501 7.91 mm to (139.5, 89.5), turned to 0 degrees
- moved SW601 7.91 mm to (114.5, 114.5), turned to 0 degrees
- moved SW701 7.91 mm to (139.5, 114.5), turned to 0 degrees
