File: Kicad/NiController/NiController_ledRing4.kicad_pcb (KiCad board)
At the start: 2 copper layers, 50 x 50 mm, 130 parts, among them J601 Conn_01x03, J602 Conn_01x03

Commit message: enc btn
Parts:
- moved J601 0.38 mm to (104.1, 124.1)
- moved J602 0.38 mm to (149.9, 124.1)
Routing:
- net +5V: track 85.0 -> 96.0 mm, vias 8 -> 14
- net /ledRing4/ledRing2/DOUT: track 45.6 -> 45.7 mm, vias 0 -> 2
- net GND: vias 54 -> 119
Other:
- outline, holes or cut-outs redrawn

Commit message: main
Parts:
- J601, J602: moved to B.Cu
- turned J601 to 180 degrees
- turned J602 to 180 degrees
