File: Kicad/NiController/encoder.kicad_sch (KiCad schematic)
At the start: 4 parts, among them SW401 RotaryEncoder_Switch

Commit message: main
Parts:
- SW401: footprint Rotary_Encoder:RotaryEncoder_Bourns_Vertical_PEC12R-3x17F-Sxxxx -> NiLibrary:PEC11-4xxxF-Sxxxx
Changed lines of the file:
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@@
 			)
 		)
-		(property "Footprint" "Rotary_Encoder:RotaryEncoder_Bourns_Vertical_PEC12R-3x17F-Sxxxx"
+		(property "Footprint" "NiLibrary:PEC11-4xxxF-Sxxxx"
 			(at 72.39 46.736 0)
 			(effects
