File: Kicad/NiController/main.kicad_sch (KiCad schematic)
At the start: 13 parts, among them J201 Barrel_Jack_Switch, J202 Conn_01x02, J203 Conn_01x02, J204 Conn_01x06_Socket, J205 Conn_01x06_Socket, Q201 Q_PMOS_GDS

Commit message: main
Parts:
- removed C202: 1u, Capacitor_SMD:C_0603_1608Metric, symbol Device:C_Small
- removed J204, J205: Conn_01x06_Socket, Connector_PinSocket_2.54mm:PinSocket_1x06_P2.54mm_Vertical, symbol Connector:Conn_01x06_Socket
- added J204: Conn_01x04, Connector_PinSocket_2.54mm:PinSocket_1x04_P2.54mm_Vertical, symbol Connector_Generic:Conn_01x04
- added J205: USB_C_Receptacle_USB2.0_16P, Connector_USB:USB_C_Receptacle_G-Switch_GT-USB-7010ASV, symbol Connector:USB_C_Receptacle_USB2.0_16P
- added R201, R202: 5.1k, Resistor_SMD:R_0603_1608Metric, symbol Device:R_Small
- added U201: ~, NiLibrary:AE-MYMGK00506ERSR-5V0, symbol NiLibrary:AE-MYMGK00506ERSR-5V0
Connections:
- net +5V: now also U201.7 (VOUT), U201.8 (VOUT), U201.9 (VOUT)
- net GND: now also J204.1 (Pin_1), J205.A1 (GND), J205.A12 (GND), J205.B1 (GND), J205.B12 (GND), J205.S1 (SHIELD), R201.2, R202.2, U201.10 (GND), U201.11 (GND), U201.12 (GND), U201.3 (GND), U201.4 (GND)
- net VAUX: now also U201.5 (VIN), U201.6 (VIN)
- new net: J205.A5 (CC1), R202.1
- new net: J205.B5 (CC2), R201.1
- new net D+: J204.2 (Pin_2), J205.A6 (D+), J205.B6 (D+)
- new net D-: J204.3 (Pin_3), J205.A7 (D-), J205.B7 (D-)
- new net VBUS: J204.4 (Pin_4), J205.A4 (VBUS), J205.A9 (VBUS), J205.B4 (VBUS), J205.B9 (VBUS)
