File: Kicad/NiController/NiController_main.kicad_pcb (KiCad board)
At the start: 2 copper layers, 27 parts, among them J201 Barrel_Jack_Switch, J202 Conn_01x02, J203 Conn_01x02, J205 Conn_01x06_Socket, J206 Conn_01x06_Socket, J301 Conn_02x09_Odd_Even, J302 Conn_02x09_Odd_Even, J303 Conn_02x03_Odd_Even, J304 Conn_02x03_Odd_Even, J305 RJ45_Hanrun_HR911105A_Horizon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, Q201 Q_PMOS_GDS, U301 Teensy4.1, U302 74LVC1GU04, U303 MCP23S17_SS, U304 MCP23S17_SS

Commit message: main
Parts:
- removed C206: 1u, Capacitor_SMD:C_0603_1608Metric
- removed the C302 at (198.0, 99.4)
- removed C303: 100n, Capacitor_SMD:C_0603_1608Metric
- removed J206: Conn_01x06_Socket, Connector_PinSocket_2.54mm:PinSocket_1x06_P2.54mm_Vertical
- removed the J301 at (89.8, 67.0)
- removed the J302 at (167.3, 56.8)
- removed U303, U304: MCP23S17_SS, Package_SO:SSOP-28_5.3x10.2mm_P0.65mm
- added C401: 100n, Capacitor_SMD:C_0603_1608Metric, F.Cu at (-18.9, 91.9)
- added C501: 100n, Capacitor_SMD:C_0603_1608Metric, F.Cu at (-18.9, 54.8)
- added C601: 100n, Capacitor_SMD:C_0603_1608Metric, F.Cu at (5.65, 54.8)
- added C701: 100n, Capacitor_SMD:C_0603_1608Metric, F.Cu at (30.2, 54.8)
- added J204: Conn_01x04, Connector_PinSocket_2.54mm:PinSocket_1x04_P2.54mm_Vertical, F.Cu at (73.3, 135.6)
- added J304: Conn_02x03_Odd_Even, Connector_PinSocket_2.54mm:PinSocket_2x03_P2.54mm_Vertical, F.Cu at (28.1, 81.0)
- added J305: Conn_02x03_Odd_Even, Connector_PinSocket_2.54mm:PinSocket_2x03_P2.54mm_Vertical, F.Cu at (35.2, 81.0)
- added J401: Conn_02x10_Odd_Even, Connector_IDC:IDC-Header_2x10_P2.54mm_Vertical, F.Cu at (69.5, 65.7)
- added J501: Conn_02x10_Odd_Even, Connector_IDC:IDC-Header_2x10_P2.54mm_Vertical, F.Cu at (-27.6, 47.6)
- added J601: Conn_02x10_Odd_Even, Connector_IDC:IDC-Header_2x10_P2.54mm_Vertical, F.Cu at (-3.10, 47.6)
- added J701: Conn_02x10_Odd_Even, Connector_IDC:IDC-Header_2x10_P2.54mm_Vertical, F.Cu at (21.4, 47.6)
- added R201: 5.1k, Resistor_SMD:R_0603_1608Metric, F.Cu at (80.5, 140.6)
- added R202: 5.1k, Resistor_SMD:R_0603_1608Metric, F.Cu at (73.8, 140.6)
- added U201: ~, NiLibrary:AE-MYMGK00506ERSR-5V0, F.Cu at (60.6, 112.7)
- added U401: MCP23S17_SS, Package_SO:SSOP-28_5.3x10.2mm_P0.65mm, F.Cu at (58.3, 88.3)
- added U501: MCP23S17_SS, Package_SO:SSOP-28_5.3x10.2mm_P0.65mm, F.Cu at (84.8, 88.6)
- added U601: MCP23S17_SS, Package_SO:SSOP-28_5.3x10.2mm_P0.65mm, F.Cu at (8.92, 47.5)
- added U701: MCP23S17_SS, Package_SO:SSOP-28_5.3x10.2mm_P0.65mm, F.Cu at (33.5, 47.5)
- J205: value Conn_01x06_Socket -> USB_C_Receptacle_USB2.0_16P; footprint Connector_PinSocket_2.54mm:PinSocket_1x06_P2.54mm_Vertical -> Connector_USB:USB_C_Receptacle_G-Switch_GT-USB-7010ASV
- moved U302 48.6 mm to (107.9, 74.0)
- moved J301 34.7 mm to (89.2, 136.6)
- moved U301 12.8 mm to (101.3, 112.7)
- moved J205 5.08 mm to (77.1, 147.2), turned to 0 degrees
- moved Q201 3.81 mm to (59.4, 132.8)
- moved J201 2.03 mm to (62.2, 141.0)
- renumbered C304 to C302, J305 to J301, J303 to J302, J304 to J303
Connections:
- J303 pad 4: unconnected-(J304-Pin_4-Pad4) -> Net-(J303-Pin_4)
- U301 pad 46: /main/Teensy/3.3V -> +3V3

Commit message: main
Parts:
- J302, J303, J304, J305: footprint Connector_PinSocket_2.54mm:PinSocket_2x03_P2.54mm_Vertical -> Connector_IDC:IDC-Header_2x03_P2.54mm_Vertical; moved to B.Cu
- J401, J501, J601, J701: moved to B.Cu
- moved J501 146.9 mm to (118.4, 63.2), turned to 180 degrees
- moved C201 128.9 mm to (53.5, 131.1)
- moved D201 127.2 mm to (59.4, 141.3), turned to -90 degrees
- moved C501 117.6 mm to (89.2, 101.3)
- moved C601 112.6 mm to (108.3, 101.3)
- moved C301 112.3 mm to (86.7, 111.4), turned to 180 degrees
- moved C701 107.7 mm to (127.3, 101.3)
- moved J202 106.8 mm to (80.1, 155.9)
- moved J203 106.8 mm to (84.8, 155.9)
- moved J303 104.1 mm to (107.0, 63.2), turned to 180 degrees
- moved R301 103.9 mm to (97.5, 133.0)
- moved U601 102.4 mm to (96.8, 100.0)
- moved J601 99.9 mm to (95.6, 63.2), turned to 180 degrees
- moved C401 89.5 mm to (70.2, 101.3)
- moved U401 77.5 mm to (134.9, 100.0), turned to 0 degrees
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Connections:
- C401 pad 2: /main/Teensy/Mcp23S17_0/3.3V -> +3V3
- C501 pad 2: /main/Teensy/Mcp23S17_1/3.3V -> +3V3
- C601 pad 2: /main/Teensy/Mcp23S17_2/3.3V -> +3V3
- C701 pad 2: /main/Teensy/Mcp23S17_3/3.3V -> +3V3
- U401 pad 9: /main/Teensy/Mcp23S17_0/3.3V -> +3V3
- U501 pad 9: /main/Teensy/Mcp23S17_1/3.3V -> +3V3
- U601 pad 9: /main/Teensy/Mcp23S17_2/3.3V -> +3V3
- U701 pad 9: /main/Teensy/Mcp23S17_3/3.3V -> +3V3
Routing:
- net /main/Teensy/NEOPIXEL_DATA_5V: track 0.00 -> 131.7 mm
- net +5V: track 0.00 -> 92.6 mm
- net /main/Teensy/MCP_CS: track 0.00 -> 73.0 mm
- net /main/Teensy/MCP_MISO: track 0.00 -> 67.8 mm
- net /main/Teensy/MCP_MOSI: track 0.00 -> 64.3 mm
- net /main/Teensy/MCP_SCK: track 0.00 -> 50.7 mm
- net /main/Teensy/ETH_LED: track 0.00 -> 43.7 mm, vias 0 -> 3
- net /main/Teensy/Mcp23S17_3/GPA0: track 0.00 -> 43.7 mm
- net /main/Teensy/Mcp23S17_0/GPB7: track 0.00 -> 43.2 mm
- net /main/Teensy/Mcp23S17_3/GPB7: track 0.00 -> 42.5 mm
- net /main/Teensy/Mcp23S17_2/GPA0: track 0.00 -> 42.5 mm
- net /main/Teensy/Mcp23S17_1/GPB7: track 0.00 -> 41.9 mm
- net /main/Teensy/Mcp23S17_0/GPA0: track 0.00 -> 41.7 mm
- net /main/Teensy/ETH_R+: track 0.00 -> 41.4 mm
- net /main/Teensy/Mcp23S17_2/GPB7: track 0.00 -> 40.8 mm
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