File: Kicad/NiController/mcp23s17.kicad_sch (KiCad schematic)
At the start: 3 parts, among them J401 Conn_02x10_Odd_Even, U401 MCP23S17_SS

Commit message: main
Connections:
- net 3.3V renamed +3V3
Changed lines of the file:
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@@
-		)
-	)
-	(label "3.3V"
-		(at 54.61 29.21 0)
-		(effects
-			(font
-				(size 1.27 1.27)
-			)
-			(justify left bottom)
 		)
 	)
@@
 					(unit 1)
 				)
+			)
+		)
+	)
+	(symbol
+		(lib_id "power:+3V3")
+		(at 54.61 29.21 0)
+		(unit 1)
+		(exclude_from_sim no)
+		(in_bom yes)
+		(on_board yes)
+		(dnp no)
+		(fields_autoplaced yes)
+		(property "Reference" "#PWR0322"
+			(at 54.61 33.02 0)
+			(effects
+				(font
+					(size 1.27 1.27)
+				)
+				(hide yes)
+			)
+		)
+		(property "Value" "+3V3"
+			(at 54.61 24.13 0)
+			(effects
+				(font
+					(size 1.27 1.27)
+				)
+			)
+		)
+		(property "Footprint" ""
+			(at 54.61 29.21 0)
+			(effects
+				(font
+					(size 1.27 1.27)
+				)
+				(hide yes)
+			)
+		)
+		(property "Datasheet" ""
+			(at 54.61 29.21 0)
+			(effects
+				(font
+					(size 1.27 1.27)
+				)
+				(hide yes)
+			)
+		)
+		(property "Description" "Power symbol creates a global label with name \"+3V3\""
+			(at 54.61 29.21 0)
+			(effects
+				(font
+					(size 1.27 1.27)
+				)
+				(hide yes)
+			)
+		)
+		(pin "1"
+		)
+		(instances
+			(project "NiController_main"
+				(path "/e70b5343-6e83-46b0-b96e-745e0612c526/9a27d9c3-2260-4575-8c04-ae473aff735e/0ec8e54a-6fc3-442d-ab20-7305dd2533aa/15c85ce5-3ae2-4f01-8b90-8ea1c8076173"
+					(reference "#PWR0323")
+					(unit 1)
+				)
+				(path "/e70b5343-6e83-46b0-b96e-745e0612c526/9a27d9c3-2260-4575-8c04-ae473aff735e/0ec8e54a-6fc3-442d-ab20-7305dd2533aa/48cb3e10-8f3c-4c7b-bf1e-6a45780257dc"
+					(reference "#PWR0322")
+					(unit 1)
+				)
+				(path "/e70b5343-6e83-46b0-b96e-745e0612c526/9a27d9c3-2260-4575-8c04-ae473aff735e/0ec8e54a-6fc3-442d-ab20-7305dd2533aa/49917f19-3dd3-46f0-b3af-d86354fee2d9"
+					(reference "#PWR0324")
+					(unit 1)
+				)
+				(path "/e70b5343-6e83-46b0-b96e-745e0612c526/9a27d9c3-2260-4575-8c04-ae473aff735e/0ec8e54a-6fc3-442d-ab20-7305dd2533aa/4e2e2a40-baec-45b6-a562-a187f286ec6c"
+					(reference "#PWR0325")
+					(unit 1)
+				)
