File: Kicad/NiController/teensy.kicad_sch (KiCad schematic)
At the start: 14 parts, among them J301 RJ45_Hanrun_HR911105A_Horizon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, J302 Conn_02x09_Odd_Even, J303 Conn_02x03_Odd_Even, J304 Conn_02x03_Odd_Even, J305 Conn_02x09_Odd_Even, U301 Teensy4.1, U302 74LVC1GU04, U303 MCP23S17_SS, U304 MCP23S17_SS

Commit message: main
Parts:
- removed C303, C304: 100n, Capacitor_SMD:C_0603_1608Metric, symbol Device:C_Small
- removed J302, J305: Conn_02x09_Odd_Even, Connector_PinSocket_2.54mm:PinSocket_2x09_P2.54mm_Vertical, symbol Connector_Generic:Conn_02x09_Odd_Even
- removed U303, U304: MCP23S17_SS, Package_SO:SSOP-28_5.3x10.2mm_P0.65mm, symbol Interface_Expansion:MCP23S17_SS
- added J304, J305: Conn_02x03_Odd_Even, Connector_PinSocket_2.54mm:PinSocket_2x03_P2.54mm_Vertical, symbol Connector_Generic:Conn_02x03_Odd_Even
- renumbered J303 to J302, J304 to J303
Connections:
- net GND: now also J304.1 (Pin_1), J304.2 (Pin_2), J305.1 (Pin_1), J305.2 (Pin_2)
- net VIN: now also J304.5 (Pin_5), J304.6 (Pin_6), J305.5 (Pin_5), J305.6 (Pin_6)
- net at J303.4 (Pin_4): now also J304.3 (Pin_3)
- net 3.3V renamed +3V3
- new net: J304.4 (Pin_4), J305.3 (Pin_3)
Other:
- added sheet Mcp23S17_0 (mcp23s17.kicad_sch)
- added sheet Mcp23S17_1 (mcp23s17.kicad_sch)
- added sheet Mcp23S17_2 (mcp23s17.kicad_sch)
- added sheet Mcp23S17_3 (mcp23s17.kicad_sch)
- moved on the sheet: J302, J303

Commit message: main
Parts:
- J302, J303, J304, J305: footprint Connector_PinSocket_2.54mm:PinSocket_2x03_P2.54mm_Vertical -> Connector_IDC:IDC-Header_2x03_P2.54mm_Vertical
Changed lines of the file:
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@@
 			)
 		)
-		(property "Footprint" "Connector_PinSocket_2.54mm:PinSocket_2x03_P2.54mm_Vertical"
+		(property "Footprint" "Connector_IDC:IDC-Header_2x03_P2.54mm_Vertical"
 			(at 196.215 81.915 0)
 			(effects
@@
 			)
 		)
-		(property "Footprint" "Connector_PinSocket_2.54mm:PinSocket_2x03_P2.54mm_Vertical"
+		(property "Footprint" "Connector_IDC:IDC-Header_2x03_P2.54mm_Vertical"
 			(at 196.215 102.235 0)
 			(effects
@@
 			)
 		)
-		(property "Footprint" "Connector_PinSocket_2.54mm:PinSocket_2x03_P2.54mm_Vertical"
+		(property "Footprint" "Connector_IDC:IDC-Header_2x03_P2.54mm_Vertical"
 			(at 196.215 120.65 0)
 			(effects
@@
 			)
 		)
-		(property "Footprint" "Connector_PinSocket_2.54mm:PinSocket_2x03_P2.54mm_Vertical"
+		(property "Footprint" "Connector_IDC:IDC-Header_2x03_P2.54mm_Vertical"
 			(at 196.215 138.43 0)
 			(effects
